Commit message: modified xacro to simulate fanuc workcell, z position of frames may need some tweaking

File: snp_support/urdf/workcell.xacro (robot description, xacro)
@@ -13,9 +13,9 @@
   <link name="world"/>
   <!-- Add Floor -->
-  <xacro:property name="length" value="9.0"/>
-  <xacro:property name="width" value="6.0"/>
+  <xacro:property name="length" value="1.1176"/>
+  <xacro:property name="width" value="1.4732"/>
   <link name="floor">
     <visual>
-      <origin xyz="0 -${width/10} 0.001" rpy="0 0 0"/>
+      <origin xyz="0 -${0/10} 0.001" rpy="0 0 0"/>
       <geometry>
         <box size="${length} ${width} 0.001"/>
@@ -23,5 +23,5 @@
     </visual>
     <collision>
-      <origin xyz="0 -${width/10} 0.001" rpy="0 0 0"/>
+      <origin xyz="0 -${0/10} 0.001" rpy="0 0 0"/>
       <geometry>
         <box size="${length} ${width} 0.001"/>
@@ -34,32 +34,30 @@
     <child link="floor"/>
   </joint>
-  <!-- Add table -->
-  <link name="table">
+  <!-- Add ceiling -->
+  <xacro:property name="length" value="1.1176"/>
+  <xacro:property name="width" value="1.4732"/>
+  <link name="ceiling">
     <visual>
+      <origin xyz="0 -${0/10} 0.001" rpy="0 0 0"/>
       <geometry>
-        <mesh filename="package://snp_support/meshes/visual/steel_table.ply"/>
+        <box size="${length} ${width} 0.001"/>
       </geometry>
-      <material name="dark_gray"/>
     </visual>
     <collision>
+      <origin xyz="0 -${0/10} 0.001" rpy="0 0 0"/>
       <geometry>
-        <mesh filename="package://snp_support/meshes/collision/steel_table.ply"/>
-      </geometry>
-    </collision>
-    <collision>
-      <origin xyz="0 0 0.726" rpy="0 0 0"/>
-      <geometry>
-        <box size="1.9 0.95 0.05"/>
+        <box size="${length} ${width} 0.001"/>
       </geometry>
     </collision>
   </link>
-  <joint name="floor_to_table" type="fixed">
+  <joint name="floor_to_ceiling" type="fixed">
     <parent link="floor"/>
-    <child link="table"/>
+    <child link="ceiling"/>
+    <origin xyz="0 0 1.1049" rpy="0 0 0"/>
   </joint>
-  <joint name="table_to_base" type="fixed">
-    <parent link="table"/>
+  <joint name="ceiling_to_base" type="fixed">
+    <parent link="ceiling"/>
     <child link="base_link"/>
-    <origin xyz="-0.61 0 0.723" rpy="0 0 0"/>
+    <origin xyz="-0.37465 -0.1524 0" rpy="0 -3.14 -3.14"/>
   </joint>
   <!-- Create a frame representing the robot tool flange (behind the teach tool and nominal tool0 frame) for IKFast -->

Commit message: Added phone mesh with Tyler's help, troubleshooting ply and stl from Solidworks

File: snp_support/urdf/workcell.xacro (robot description, xacro)
@@ -71,5 +71,5 @@
   </joint>
   <!-- Add End Effector Components -->
-  <link name="ee">
+  <!--<link name="ee">
     <visual>
       <geometry>
@@ -121,5 +121,5 @@
     <parent link="tool0"/>
     <child link="ee"/>
-  </joint>
+  </joint>-->
   <xacro:property name="camera_cal" value="${load_yaml('$(find snp_support)/config/camera_calibration.yaml')}" />
   <link name="camera_color_optical_frame"/>

Commit message: Added phone mesh with Tyler's help, troubleshooting ply and stl from Solidworks

File: snp_support/urdf/workcell.xacro (robot description, xacro)
@@ -69,5 +69,5 @@
   </joint>
   <!-- Add End Effector Components -->
-  <link name="ee">
+  <!--<link name="ee">
     <visual>
       <geometry>
@@ -119,5 +119,5 @@
     <parent link="tool0"/>
     <child link="ee"/>
-  </joint>
+  </joint>-->
   <xacro:property name="camera_cal" value="${load_yaml('$(find snp_support)/config/camera_calibration.yaml')}" />
   <link name="camera_color_optical_frame"/>

Commit message: Phone mesh is on floor and primative end effector is added to urdf. Need to offset end effector from tool0 so that it doesnt clip into the robot

File: snp_support/urdf/workcell.xacro (robot description, xacro)
@@ -69,5 +69,25 @@
   </joint>
   <!-- Add End Effector Components -->
-  <!--<link name="ee">
+  <xacro:property name="ee_length" value="0.254"/> <!--10 in converted to m -->
+  <xacro:property name="ee_radius" value="0.035"/> <!--70mm is diameter of joint 6 from fanuc specs-->
+  <link name="ee">
+    <visual>
+<!--      <origin xyz="0 -${0/10} 0.001" rpy="0 0 0"/>-->
+      <geometry>
+        <cylinder length="${ee_length}" radius="${ee_radius}"/>
+      </geometry>
+    </visual>
+    <collision>
+<!--      <origin xyz="0 -${0/10} 0.001" rpy="0 0 0"/>-->
+      <geometry>
+        <cylinder length="${ee_length}" radius="${ee_radius}"/>
+      </geometry>
+    </collision>
+  </link>
+  <joint name="tool0_to_ee" type="fixed">
+    <parent link="tool0"/>
+    <child link="ee"/>
+  </joint>
+<!--<link name="ee">
     <visual>
       <geometry>

Commit message: Adjusted line_spacing, min_segment_lengt and point_spacing (lines 500-506) in /home/D10.US.SWRI.ORG/dspielman/snp/snp_ws/src/scan_n_plan_workshop/snp_application/src/rosconwindow.cpp,removed all faces on mesh except the top one, moved sand_tcp to be at the end of the end effector. Currently troubleshooting why tool path generation is broken (worked after adjusting parameters for tool path planning in rosconwindow.cpp

File: snp_support/urdf/workcell.xacro (robot description, xacro)
@@ -73,5 +73,5 @@
   <link name="ee">
     <visual>
-<!--      <origin xyz="0 -${0/10} 0.001" rpy="0 0 0"/>-->
+      <origin xyz="0 0 0.115" rpy="0 0 0"/>-->
       <geometry>
         <cylinder length="${ee_length}" radius="${ee_radius}"/>
@@ -79,5 +79,5 @@
     </visual>
     <collision>
-<!--      <origin xyz="0 -${0/10} 0.001" rpy="0 0 0"/>-->
+    <origin xyz="0 0 0.115" rpy="0 0 0"/>-->
       <geometry>
         <cylinder length="${ee_length}" radius="${ee_radius}"/>
@@ -158,7 +158,7 @@
   <link name="sand_tcp"/>
   <joint name="sand_tcp_joint" type="fixed">
-    <parent link="tool_flange"/>
+    <parent link="ee"/>
     <child link="sand_tcp"/>
-    <origin xyz="-0.26261 0 ${0.08259 + dt_flange_width}" rpy="${radians(-90)} 0 ${radians(90)}"/>
+    <origin xyz="0 0 ${ee_length}" rpy="0 0 0"/>
   </joint>
 </robot>

Commit message: Tool path planning works, motion planning broken. Working with Tyler to fix

File: snp_support/urdf/workcell.xacro (robot description, xacro)
@@ -78,10 +78,10 @@
       </geometry>
     </visual>
-    <collision>
-    <origin xyz="0 0 0.115" rpy="0 0 0"/>-->
+    <!--<collision>
+    <origin xyz="0 0 0.115" rpy="0 0 0"/>
       <geometry>
         <cylinder length="${ee_length}" radius="${ee_radius}"/>
       </geometry>
-    </collision>
+    </collision>-->
   </link>
   <joint name="tool0_to_ee" type="fixed">
@@ -156,9 +156,15 @@
   </joint>
   <!-- Add TCP -->
+  <link name="sand_tcp_1"/>
+  <joint name="sand_tcp_1_joint" type="fixed">
+    <parent link="ee"/>
+    <child link="sand_tcp_1"/>
+    <origin xyz="0 0 ${ee_length}" rpy="0 0 0"/>
+  </joint>
   <link name="sand_tcp"/>
   <joint name="sand_tcp_joint" type="fixed">
-    <parent link="ee"/>
+    <parent link="sand_tcp_1"/>
     <child link="sand_tcp"/>
-    <origin xyz="0 0 ${ee_length}" rpy="0 0 0"/>
+    <origin xyz="0 0 0" rpy="3.14 0 0"/>
   </joint>
 </robot>

Commit message: Motion plan works, mesh was offset

File: snp_support/urdf/workcell.xacro (robot description, xacro)
@@ -156,15 +156,9 @@
   </joint>
   <!-- Add TCP -->
-  <link name="sand_tcp_1"/>
+  <link name="sand_tcp"/>
   <joint name="sand_tcp_1_joint" type="fixed">
     <parent link="ee"/>
-    <child link="sand_tcp_1"/>
+    <child link="sand_tcp"/>
     <origin xyz="0 0 ${ee_length}" rpy="0 0 0"/>
   </joint>
-  <link name="sand_tcp"/>
-  <joint name="sand_tcp_joint" type="fixed">
-    <parent link="sand_tcp_1"/>
-    <child link="sand_tcp"/>
-    <origin xyz="0 0 0" rpy="3.14 0 0"/>
-  </joint>
 </robot>

Commit message: Updated urdf of fanuc robot to include workcell walls

File: snp_support/urdf/workcell.xacro (robot description, xacro)
@@ -6,13 +6,19 @@
   <!-- Add World -->
   <material name="light_gray">
-    <color rgba="0.7 0.7 0.7 1"/>
+    <color rgba="0.7 0.7 0.7 0.5"/>
   </material>
   <material name="dark_gray">
     <color rgba="0.3 0.3 0.3 1"/>
   </material>
+  <material name="blue">
+    <color rgba="0 0 1 1"/>
+  </material>
+  <material name="black">
+    <color rgba="0 0 0 1"/>
+  </material>
   <link name="world"/>
   <!-- Add Floor -->
-  <xacro:property name="length" value="1.1176"/>
-  <xacro:property name="width" value="1.4732"/>
+  <xacro:property name="length" value="1.171575"/>
+  <xacro:property name="width" value="0.936625"/>
   <link name="floor">
     <visual>
@@ -21,4 +27,5 @@
         <box size="${length} ${width} 0.001"/>
       </geometry>
+      <material name="light_gray"/>
     </visual>
     <collision>
@@ -34,13 +41,102 @@
     <child link="floor"/>
   </joint>
+    <!-- Add Walls for Collision -->
+    <xacro:property name="lengthw" value="1.171575"/>
+    <xacro:property name="widthw" value="1.11125"/>
+    <!-- Right Wall -->
+    <link name="wall_right">
+      <visual>
+        <origin xyz="0.0508 -${width/2+0.01905} ${0.001+widthw/2}" rpy="${pi/2} 0 0"/>
+        <geometry>
+          <box size="${lengthw-0.0508} ${widthw} 0.001"/>
+        </geometry>
+        <material name="light_gray"/>
+      </visual>
+      <collision>
+        <origin xyz="0.0508 -${width/2+0.01905} ${0.001+widthw/2}" rpy="${pi/2} 0 0"/>
+        <geometry>
+          <box size="${lengthw-0.0508} ${widthw} 0.001"/>
+        </geometry>
+      </collision>
+    </link>
+    <joint name="floor_to_wall_right" type="fixed">
+      <origin xyz="0 0 0" rpy="0 0 0"/>
+      <parent link="floor"/>
+      <child link="wall_right"/>
+    </joint>
+    <!-- Back Wall -->
+    <link name="wall_back">
+      <visual>
+        <origin xyz="${length/2+0.009525} 0 ${0.001+widthw/2}" rpy="${pi/2} 0 ${pi/2}"/>
+        <geometry>
+          <box size="${width} ${widthw} 0.001"/>
+        </geometry>
+        <material name="light_gray"/>
+      </visual>
+      <collision>
+        <origin xyz="${length/2+0.009525} 0 ${0.001+widthw/2}" rpy="${pi/2} 0 ${pi/2}"/>
+        <geometry>
+          <box size="${width} ${widthw} 0.001"/>
+        </geometry>
+      </collision>
+    </link>
+    <joint name="floor_to_wall_back" type="fixed">
+      <origin xyz="0 0 0" rpy="0 0 0"/>
+      <parent link="floor"/>
+      <child link="wall_back"/>
+    </joint>
+    <!-- Front Wall -->
+    <link name="wall_front">
+      <visual>
+        <origin xyz="-${length/2-0.0762} 0 ${0.001+widthw/2}" rpy="${pi/2} 0 ${pi/2}"/>
+        <geometry>
+          <box size="${width} ${widthw} 0.001"/>
+        </geometry>
+        <material name="light_gray"/>
+      </visual>
+      <collision>
+      <origin xyz="-${length/2-0.0762} 0 ${0.001+widthw/2}" rpy="${pi/2} 0 ${pi/2}"/>
+        <geometry>
+          <box size="${width} ${widthw} 0.001"/>
+        </geometry>
+      </collision>
+    </link>
+    <joint name="floor_to_wall_front" type="fixed">
+      <origin xyz="0 0 0" rpy="0 0 0"/>
+      <parent link="floor"/>
+      <child link="wall_front"/>
+    </joint>
+  <!-- Add Acryllic-->
+    <xacro:property name="lengtha" value="0.923925"/>
+    <xacro:property name="widtha" value="0.8763"/>black
+    <xacro:property name="thicknessa_plus_p" value="${0.01+0.0047625}"/>
+    <link name="acryllic">
+      <visual>
+        <origin xyz="0 0 ${0.001+thicknessa_plus_p/2}"/>
+        <geometry>
+          <box size="${lengtha} ${widtha} ${thicknessa_plus_p}"/>
+        </geometry>
+        <material name="blue"/>
+      </visual>
+      <collision>
+        <origin xyz="0 -${0/10} 0.001" rpy="0 0 0"/>
+        <geometry>
+          <box size="${lengtha} ${widtha} ${0.001+thicknessa_plus_p/2}"/>
+        </geometry>
+      </collision>
+    </link>
+    <joint name="floor_to_acryllic" type="fixed">
+      <origin xyz="-0.02225 0.004775 0" rpy="0 0 0"/>
+      <parent link="floor"/>
+      <child link="acryllic"/>
+    </joint>
   <!-- Add ceiling -->
-  <xacro:property name="length" value="1.1176"/>
-  <xacro:property name="width" value="1.4732"/>
   <link name="ceiling">
     <visual>
-      <origin xyz="0 -${0/10} 0.001" rpy="0 0 0"/>
-      <geometry>
-        <box size="${length} ${width} 0.001"/>
-      </geometry>
+      <origin xyz="0.0508 -${0/10} 0.001" rpy="0 0 0"/>
+      <geometry>3.3125+7.375/2
+        <box size="${length-0.0508} ${width} 0.001"/>
+      </geometry>
+      <material name="black"/>
     </visual>
     <collision>
@@ -54,10 +150,10 @@
     <parent link="floor"/>
     <child link="ceiling"/>
-    <origin xyz="0 0 1.1049" rpy="0 0 0"/>
+    <origin xyz="0 0 1.11125" rpy="0 0 0"/>
   </joint>
   <joint name="ceiling_to_base" type="fixed">
     <parent link="ceiling"/>
     <child link="base_link"/>
-    <origin xyz="-0.37465 -0.1524 0" rpy="0 -3.14 -3.14"/>
+    <origin xyz="-${length/2-2*0.0508-0.1778} -0.169135 0" rpy="0 -3.14 -3.14"/>
   </joint>
   <!-- Create a frame representing the robot tool flange (behind the teach tool and nominal tool0 frame) for IKFast -->
@@ -77,11 +173,12 @@
         <cylinder length="${ee_length}" radius="${ee_radius}"/>
       </geometry>
-    </visual>
-    <!--<collision>
-    <origin xyz="0 0 0.115" rpy="0 0 0"/>
+      <material name="black"/>
+    </visual>
+    <collision>
+      <origin xyz="0 0 0.115" rpy="0 0 0"/>
       <geometry>
         <cylinder length="${ee_length}" radius="${ee_radius}"/>
       </geometry>
-    </collision>-->
+    </collision>
   </link>
   <joint name="tool0_to_ee" type="fixed">
@@ -140,5 +237,5 @@
     <child link="ee"/>
   </joint>-->
-  <xacro:property name="camera_cal" value="${load_yaml('$(find snp_support)/config/camera_calibration.yaml')}" />
+ <!-- <xacro:property name="camera_cal" value="${load_yaml('$(find snp_support)/config/camera_calibration.yaml')}" />
   <link name="camera_color_optical_frame"/>
   <joint name="tool0_to_camera" type="fixed">
@@ -154,5 +251,5 @@
     <origin xyz="${camera_cal['target_mount_to_target_pos']['x']} ${camera_cal['target_mount_to_target_pos']['y']} ${camera_cal['target_mount_to_target_pos']['z']}"
             rpy="${camera_cal['target_mount_to_target_rpy']['x']} ${camera_cal['target_mount_to_target_rpy']['y']} ${camera_cal['target_mount_to_target_rpy']['z']}" />
-  </joint>
+  </joint>-->
   <!-- Add TCP -->
   <link name="sand_tcp"/>

Commit message: update workcell.xacro with end-effector visual and collison model and sand_tcp frame, mesh files included.

File: snp_support/urdf/workcell.xacro (robot description, xacro)
@@ -155,5 +155,5 @@
     <parent link="ceiling"/>
     <child link="base_link"/>
-    <origin xyz="-${length/2-2*0.0508-0.1778} -0.169135 0" rpy="0 -3.14 -3.14"/>
+    <origin xyz="-${length/2-2*0.0508-0.1778} -0.169135 0" rpy="0 -3.14 1.5708"/>
   </joint>
   <!-- Create a frame representing the robot tool flange (behind the teach tool and nominal tool0 frame) for IKFast -->
@@ -169,14 +169,14 @@
   <link name="ee">
     <visual>
-      <origin xyz="0 0 0.115" rpy="0 0 0"/>-->
-      <geometry>
-        <cylinder length="${ee_length}" radius="${ee_radius}"/>
+      <origin xyz="0 0 0" rpy="0 0 0"/>-->
+      <geometry>
+        <mesh filename="package://snp_support/meshes/visual/end_effector_viz.ply"/>
       </geometry>
       <material name="black"/>
     </visual>
     <collision>
-      <origin xyz="0 0 0.115" rpy="0 0 0"/>
-      <geometry>
-        <cylinder length="${ee_length}" radius="${ee_radius}"/>
+      <origin xyz="0 0 0" rpy="0 0 0"/>
+      <geometry>
+        <mesh filename="package://snp_support/meshes/collision/end_effector_convhull.ply"/>
       </geometry>
     </collision>
@@ -185,4 +185,5 @@
     <parent link="tool0"/>
     <child link="ee"/>
+    <origin xyz="0 0 0" rpy="-1.5708 0 1.5708"/>
   </joint>
 <!--<link name="ee">
@@ -255,5 +256,5 @@
   <link name="sand_tcp"/>
   <joint name="sand_tcp_1_joint" type="fixed">
-    <parent link="ee"/>
+    <parent link="tool0"/>
     <child link="sand_tcp"/>
     <origin xyz="0 0 ${ee_length}" rpy="0 0 0"/>

Commit message: Point cloud now working. Used data from first camera cal to populate origin of camera link in urdf

File: snp_support/urdf/workcell.xacro (robot description, xacro)
@@ -185,5 +185,5 @@
     <parent link="tool0"/>
     <child link="ee"/>
-    <origin xyz="0 0 0" rpy="-1.5708 0 1.5708"/>
+    <origin xyz="0 0 0" rpy="1.5708 3.14 1.5708"/>
   </joint>
 <!--<link name="ee">
@@ -230,5 +230,5 @@
     <collision name="sidebracket2">
       <geometry>
-        <mesh filename="package://snp_support/meshes/collision/bracket2.ply"/>
+        <mesh filename="package://snpsupport/meshes/collision/bracket2.ply"/>
       </geometry>
     </collision>
@@ -238,5 +238,5 @@
     <child link="ee"/>
   </joint>-->
- <!-- <xacro:property name="camera_cal" value="${load_yaml('$(find snp_support)/config/camera_calibration.yaml')}" />
+ <xacro:property name="camera_cal" value="${load_yaml('$(find snp_support)/config/camera_calibration.yaml')}" />
   <link name="camera_color_optical_frame"/>
   <joint name="tool0_to_camera" type="fixed">
@@ -246,5 +246,5 @@
             rpy="${camera_cal['camera_mount_to_camera_rpy']['x']} ${camera_cal['camera_mount_to_camera_rpy']['y']} ${camera_cal['camera_mount_to_camera_rpy']['z']}" />
   </joint>
-  <link name="cal_target_frame"/>
+  <!-- <link name="cal_target_frame"/>
   <joint name="target_mount_to_target" type="fixed">
     <parent link="base_link"/>
