Commit message: wip to add table to the workspace xacro

File: snp_blending/urdf/mh180_120/mh180_120_macro.xacro (robot description, xacro)
@@ -123,5 +123,5 @@
     <!-- end of link list -->
     <!-- joint list -->
-    <joint name="${prefix}joint_1" type="revolute">
+    <joint name="${prefix}joint_1_s" type="revolute">
       <origin xyz="0 0 0.650" rpy="0 0 0"/>
       <parent link="${prefix}base_link"/>
@@ -130,5 +130,5 @@
       <limit lower="-${radians(180)}" upper="${radians(180)}" effort="0" velocity="${radians(125)}"/>
     </joint>
-    <joint name="${prefix}joint_2" type="revolute">
+    <joint name="${prefix}joint_2_l" type="revolute">
       <origin xyz="0.325 0 0" rpy="0 0 0"/>
       <parent link="${prefix}link_s"/>
@@ -137,5 +137,5 @@
       <limit lower="-${radians(60)}" upper="${radians(76)}" effort="0" velocity="${radians(115)}"/>
     </joint>
-    <joint name="${prefix}joint_3" type="revolute">
+    <joint name="${prefix}joint_3_u" type="revolute">
       <origin xyz="0 0 1.150" rpy="0 0 0"/>
       <parent link="${prefix}link_l"/>
@@ -144,5 +144,5 @@
       <limit lower="-${radians(85)}" upper="${radians(90)}" effort="0" velocity="${radians(125)}"/>
     </joint>
-    <joint name="${prefix}joint_4" type="revolute">
+    <joint name="${prefix}joint_4_r" type="revolute">
       <origin xyz="0 0 0.3" rpy="0 0 0"/>
       <parent link="${prefix}link_u"/>
@@ -151,5 +151,5 @@
       <limit lower="-${radians(360)}" upper="${radians(360)}" effort="0" velocity="${radians(182)}"/>
     </joint>
-    <joint name="${prefix}joint_5" type="revolute">
+    <joint name="${prefix}joint_5_b" type="revolute">
       <origin xyz="1.590 0 0" rpy="0 0 0"/>
       <parent link="${prefix}link_r"/>
@@ -158,5 +158,5 @@
       <limit lower="-${radians(130)}" upper="${radians(130)}" effort="0" velocity="${radians(175)}"/>
     </joint>
-    <joint name="${prefix}joint_6" type="revolute">
+    <joint name="${prefix}joint_6_t" type="revolute">
       <origin xyz="0.225 0 0" rpy="0 0 0"/>
       <parent link="${prefix}link_b"/>
@@ -165,5 +165,5 @@
       <limit lower="-${radians(360)}" upper="${radians(360)}" effort="0" velocity="${radians(265)}"/>
     </joint>
-    <joint name="${prefix}joint_6-tool0" type="fixed">
+    <joint name="${prefix}joint_6_t-tool0" type="fixed">
       <origin xyz="0 0 0" rpy="0 ${radians(90)} 0"/>
       <parent link="${prefix}link_t"/>

File: snp_blending/urdf/workcell.xacro (robot description, xacro)
@@ -94,8 +94,13 @@
   <xacro:property name="control_boxes_width" value="${38*0.0254}"/>
   <xacro:property name="control_boxes_length" value="${130*0.0254}"/>
-  <xacro:property name="table_height" value="${33.875*0.0254}"/>
-  <xacro:property name="table_width" value="${48*0.0254}"/>
-  <xacro:property name="table_length" value="${30*0.0254}"/>
+  <xacro:property name="table_height" value="${37*0.0254}"/>
+  <xacro:property name="table_width" value="${60*0.0254}"/>
+  <xacro:property name="table_length" value="${36*0.0254}"/>
   <link name="floor"/>
+  <link name="table_temp_link">
+    <geometry>
+      <mesh filename="package://snp_blending/meshes/pushcorp/pushcorp_base.dae"/>
+    </geometry>
+  </link>
   <link name="platform">
     <visual>
@@ -217,3 +222,29 @@
     <origin xyz="-${robot_mount_width/2 + 2*0.0254 + pushcorp_box_length/2} ${robot_mount_width/2 + 17*0.0254 + pushcorp_box_width/2} ${14*0.0254 + pushcorp_box_height/2}" rpy="0 0 0"/>
   </joint>
+  <xacro:property name="table_cal" value="${load_yaml('$(find snp_blending)/config/table_calibration.yaml')}" />
+  <link name="table">
+    <visual>
+      <geometry>
+           <box size = "${table_length} ${table_width} ${table_height}"/>
+      </geometry>
+      <material name="light_gray"/>
+    </visual>
+    <collision>
+      <geometry>
+           <box size = "${table_length} ${table_width} ${table_height}"/>
+      </geometry>
+    </collision>
+  </link>
+  <joint name="floor_to_table" type="fixed">
+    <parent link="floor"/>
+    <child link="table"/>
+    <origin xyz="${table_cal['platform_to_pushcorp_base_pos']['x']} ${table_cal['platform_to_pushcorp_base_pos']['y']} ${table_cal['platform_to_pushcorp_base_pos']['z']/2}"
+            rpy="0 0 0" />
+  </joint>
+  <joint name="platform_to_pushcorp_base" type="fixed">
+    <parent link="platform"/>
+    <child link="table_temp_link"/>
+    <origin xyz="${table_cal['platform_to_pushcorp_base_pos']['x']} ${table_cal['platform_to_pushcorp_base_pos']['y']} ${table_cal['platform_to_pushcorp_base_pos']['z']/2}"
+            rpy="0 0 0" />
+  </joint>
 </robot>
