Commit message: Reorganized urdf file organization

File: snp_blending/urdf/workcell.xacro (robot description, xacro)
@@ -1,5 +1,6 @@
 <?xml version="1.0" ?>
 <robot name="motoman_mh_180_120" xmlns:xacro="http://ros.org/wiki/xacro">
-  <xacro:include filename="$(find snp_blending)/urdf/mh180_120.xacro"/>
+<xacro:include filename="$(find snp_blending)/urdf/mh180_120_macro.xacro"/>
+<xacro:motoman_mh180_120 prefix=""/>
   <material name="light_gray">
     <color rgba="0.7 0.7 0.7 1"/>
@@ -61,15 +62,18 @@
     <axis xyz="0 0 0"/>
   </joint>-->
+<xacro:property name="camera_cal" value="${load_yaml('$(find snp_automate_2022)/config/camera_calibration.yaml')}" />
   <link name="camera_color_optical_frame"/>
-  <link name="target_cal_frame"/>
-  <joint name="camera_cal_joint" type="fixed">
-    <parent link="camera_link"/>
+  <joint name="tool0_to_camera" type="fixed">
+    <parent link="tool0"/>
     <child link="camera_color_optical_frame"/>
-    <origin xyz="0.085549560652492 -0.1732631672558103 0.1329373703855808" wxyz="0.5118596229748543 -0.5074314040915237 0.4900425218487801 -0.4902768843111336"/>
-  </joint>
-  <joint name="target_cal_joint" type="fixed">
-    <parent link="floor"/>
-    <child link="target_cal_frame"/>
-    <origin xyz="0.555641489380775 0.05956001933889868 0.1229851433910979" wxyz="0.6869783604862724 -0.001114251051880176 -0.003909064875724348 -0.7266665052690842"/>
+    <origin xyz="${camera_cal['camera_mount_to_camera_pos']['x']} ${camera_cal['camera_mount_to_camera_pos']['y']} ${camera_cal['camera_mount_to_camera_pos']['z']}"
+            rpy="${camera_cal['camera_mount_to_camera_rpy']['x']} ${camera_cal['camera_mount_to_camera_rpy']['y']} ${camera_cal['camera_mount_to_camera_rpy']['z']}" />
+  </joint>
+  <link name="cal_target_frame"/>
+  <joint name="target_mount_to_target" type="fixed">
+    <parent link="base_link"/>
+    <child link="cal_target_frame"/>
+    <origin xyz="${camera_cal['target_mount_to_target_pos']['x']} ${camera_cal['target_mount_to_target_pos']['y']} ${camera_cal['target_mount_to_target_pos']['z']}"
+            rpy="${camera_cal['target_mount_to_target_rpy']['x']} ${camera_cal['target_mount_to_target_rpy']['y']} ${camera_cal['target_mount_to_target_rpy']['z']}" />
   </joint>
   <!-- TODO do we care about effort and velocity limits?-->

Commit message: Minor edits to workcell.xacro

File: snp_blending/urdf/workcell.xacro (robot description, xacro)
@@ -1,6 +1,6 @@
 <?xml version="1.0" ?>
 <robot name="motoman_mh_180_120" xmlns:xacro="http://ros.org/wiki/xacro">
-<xacro:include filename="$(find snp_blending)/urdf/mh180_120_macro.xacro"/>
-<xacro:motoman_mh180_120 prefix=""/>
+  <xacro:include filename="$(find snp_blending)/urdf/mh180_120/mh180_120_macro.xacro"/>
+  <xacro:motoman_mh180_120 prefix=""/>
   <material name="light_gray">
     <color rgba="0.7 0.7 0.7 1"/>
@@ -62,5 +62,5 @@
     <axis xyz="0 0 0"/>
   </joint>-->
-<xacro:property name="camera_cal" value="${load_yaml('$(find snp_automate_2022)/config/camera_calibration.yaml')}" />
+  <xacro:property name="camera_cal" value="${load_yaml('$(find snp_automate_2022)/config/camera_calibration.yaml')}" />
   <link name="camera_color_optical_frame"/>
   <joint name="tool0_to_camera" type="fixed">

Commit message: working preliminary scan n plan

File: snp_blending/urdf/workcell.xacro (robot description, xacro)
@@ -62,5 +62,5 @@
     <axis xyz="0 0 0"/>
   </joint>-->
-  <xacro:property name="camera_cal" value="${load_yaml('$(find snp_automate_2022)/config/camera_calibration.yaml')}" />
+  <xacro:property name="camera_cal" value="${load_yaml('$(find snp_blending)/config/camera_calibration.yaml')}" />
   <link name="camera_color_optical_frame"/>
   <joint name="tool0_to_camera" type="fixed">
@@ -97,4 +97,5 @@
   <xacro:property name="table_width" value="${60*0.0254}"/>
   <xacro:property name="table_length" value="${36*0.0254}"/>
+  <xacro:property name="table_correction" value="${5*0.0254}"/>
   <link name="floor"/>
   <link name="table_temp_link">
@@ -239,5 +240,5 @@
     <parent link="floor"/>
     <child link="table"/>
-    <origin xyz="${table_cal['platform_to_pushcorp_base_pos']['x']} ${table_cal['platform_to_pushcorp_base_pos']['y']} ${table_cal['platform_to_pushcorp_base_pos']['z']/2}"
+    <origin xyz="${table_cal['platform_to_pushcorp_base_pos']['x'] + table_width/2 - table_correction} ${table_cal['platform_to_pushcorp_base_pos']['y'] + table_length/2 - table_correction} ${table_cal['platform_to_pushcorp_base_pos']['z'] - table_height/2 - platform_height + table_correction}"
             rpy="0 0 0" />
   </joint>
@@ -245,5 +246,5 @@
     <parent link="platform"/>
     <child link="table_temp_link"/>
-    <origin xyz="${table_cal['platform_to_pushcorp_base_pos']['x']} ${table_cal['platform_to_pushcorp_base_pos']['y']} ${table_cal['platform_to_pushcorp_base_pos']['z']/2}"
+    <origin xyz="${table_cal['platform_to_pushcorp_base_pos']['x'] + table_width/2 - table_correction} ${table_cal['platform_to_pushcorp_base_pos']['y'] + table_length/2 - table_correction} ${table_cal['platform_to_pushcorp_base_pos']['z'] - table_height/2 - platform_height + table_correction}"
             rpy="0 0 0" />
   </joint>

Commit message: Added grinding tool to spindle in urdf

File: snp_blending/urdf/workcell.xacro (robot description, xacro)
@@ -33,4 +33,16 @@
       <geometry>
         <mesh filename="package://snp_blending/meshes/pushcorp/pushcorp_spindle.dae"/>
+      </geometry>
+    </collision>
+    <visual>
+      <origin xyz="0.200 ${0.19-0.01635} 0" rpy="0 ${pi/2} 0"/>
+      <geometry>
+        <cylinder radius="0.1" length="0.005"/>
+      </geometry>
+    </visual>
+    <collision>
+      <origin xyz="0.200 ${0.19-0.01635} 0" rpy="0 ${pi/2} 0"/>
+      <geometry>
+        <cylinder radius="0.1" length="0.005"/>
       </geometry>
     </collision>
@@ -182,9 +194,10 @@
     </collision>
   </link>
-  <link name="buffy_tcp"/>
+  <link name="buffy_tcp" />
   <joint name="buffy_tcp_joint" type="fixed">
     <parent link="tool0"/>
     <child link="buffy_tcp"/>
-    <origin xyz="0.292 0 0.19" rpy="0 ${pi/2} 0"/>
+<!--    <origin xyz="0.292 0 0.19" rpy="0 ${pi/2} 0"/>-->
+    <origin xyz="0.210 0 0.19" rpy="0 ${pi/2} 0"/>
   </joint>
   <joint name="floor_to_platform" type="fixed">

Commit message: Adjusted table position in urdf

File: snp_blending/urdf/workcell.xacro (robot description, xacro)
@@ -253,5 +253,5 @@
     <parent link="floor"/>
     <child link="table"/>
-    <origin xyz="${table_cal['platform_to_pushcorp_base_pos']['x'] + table_width/2 - table_correction} ${table_cal['platform_to_pushcorp_base_pos']['y'] + table_length/2 - table_correction} ${table_cal['platform_to_pushcorp_base_pos']['z'] - table_height/2 - platform_height + table_correction}"
+    <origin xyz="${table_cal['platform_to_pushcorp_base_pos']['x'] + table_width/2 - table_correction} ${table_cal['platform_to_pushcorp_base_pos']['y'] + table_length/2 - table_correction + 0.25} ${table_cal['platform_to_pushcorp_base_pos']['z'] - table_height/2 - platform_height + table_correction}"
             rpy="0 0 0" />
   </joint>
@@ -259,5 +259,5 @@
     <parent link="platform"/>
     <child link="table_temp_link"/>
-    <origin xyz="${table_cal['platform_to_pushcorp_base_pos']['x'] + table_width/2 - table_correction} ${table_cal['platform_to_pushcorp_base_pos']['y'] + table_length/2 - table_correction} ${table_cal['platform_to_pushcorp_base_pos']['z'] - table_height/2 - platform_height + table_correction}"
+    <origin xyz="${table_cal['platform_to_pushcorp_base_pos']['x'] + table_width/2 - table_correction} ${table_cal['platform_to_pushcorp_base_pos']['y'] + table_length/2 - table_correction + 0.25} ${table_cal['platform_to_pushcorp_base_pos']['z'] - table_height/2 - platform_height + table_correction}"
             rpy="0 0 0" />
   </joint>

Commit message: Updated camera calibration

File: snp_blending/urdf/workcell.xacro (robot description, xacro)
@@ -92,5 +92,5 @@
   </joint>
   <!-- Camera Calibration-->
-  <xacro:property name="camera_cal" value="${load_yaml('$(find snp_blending)/config/camera_calibration.yaml')}" />
+  <xacro:property name="camera_cal" value="${load_yaml('$(find snp_blending)/config/calibration.yaml')}" />
   <link name="camera_color_optical_frame"/>
   <joint name="tool0_to_camera" type="fixed">
